File: hw/sch_pcb/PIN_detector.kicad_sch (KiCad schematic)
At the start: 37 parts, among them Q1 2SK2394-6, U3 ISL21080DIH309, U3 SHT31-DIS, U8 OPA314, U9 AD8691

Commit message: Resolve #10
Parts:
- removed C15: 3n3, Capacitor_SMD:C_0805_2012Metric, symbol Device:C
- removed C16, C6: 100nF, Capacitor_SMD:C_0805_2012Metric, symbol Device:C
- removed C50: 10uF, Capacitor_Tantalum_SMD:CP_EIA-3216-18_Kemet-A, symbol Device:C_Polarized_Small
- removed R2: 470R, Resistor_SMD:R_0805_2012Metric, symbol Device:R
- removed R7, R9: 10k, Resistor_SMD:R_0805_2012Metric, symbol Device:R
- removed R8: 1k, Resistor_SMD:R_0805_2012Metric, symbol Device:R
- removed U9: AD8691, Package_TO_SOT_SMD:TSOT-23-5, symbol MLAB_IO:AD8691
Connections:
- net Signal: now also C10.1
Other:
- note removed: "1.2 mA"
- title: USTSIPIN03B -> USTSIPIN03C

Commit message: Update KiCAD project.
Parts:
- renumbered C17 to C19, C59 to C20, C50 to C21, C37 to C22, C5 to C25, C50 to C26, C50 to C27, C2 to C28, C24 to C29, C10 to C30, C3 to C32, C6 to C33, C50 to C34, C59 to C36, D2 to D1, R40 to R10, R14 to R12, R6 to R13, R15 to R14, R19 to R15, R22 to R16, R16 to R17, R2 to R19, R40 to R21, U3 to U10, U3 to U7
