File: hw/sch_pcb/USTSIPIN03.kicad_sch (KiCad schematic)
At the start: 8 parts, among them M1 HOLE, M2 HOLE, M3 HOLE, M4 HOLE

Commit message: Resolve #10
Other:
- title: USTSIPIN03B -> USTSIPIN03C
Changed lines of the file:
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@@
 	(paper "A4")
 	(title_block
-		(title "USTSIPIN03B")
+		(title "USTSIPIN03C")
 		(date "2024-05-30")
 		(company "kaklik <info@ust.cz>")

Commit message: Update KiCAD project.
Parts:
- renumbered FID1 to FID3, FID2 to FID4
