File: hw/sch_pcb/analogue_backend.kicad_sch (KiCad schematic)
At the start: 37 parts, among them M5 RFShield_TwoPieces, U2 AD8691, U3 ISL21080CIH341Z-TK, U3 LTC1865-MS, U4 AD8691, U5 SN74LVC2G74, U6 TS3021ILT

Commit message: Resolve #10
Other:
- title: USTSIPIN03B -> USTSIPIN03C
Changed lines of the file:
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@@
 	(paper "A4")
 	(title_block
-		(title "USTSIPIN03B")
+		(title "USTSIPIN03C")
 		(date "2023-10-23")
 		(company "kaklik <info@ust.cz>")

Commit message: Update UST_ID for ADC.
Parts:
- U3: UST_ID 651eaece462c6d9e72055763 -> 67f14385ee7fc534862c535e
Changed lines of the file:
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@@
 			)
 		)
-		(property "UST_ID" "651eaece462c6d9e72055763"
+		(property "UST_ID" "67f14385ee7fc534862c535e"
 			(at 242.57 104.14 0)
 			(effects

Commit message: Update KiCAD project.
Parts:
- renumbered C2 to C1, C59 to C12, C18 to C15, C2 to C5, C59 to C8, JP4 to JP1, R11 to R4, R11 to R5, R10 to R7, TP3 to TP1, TP3 to TP2, U3 to U1
Changed lines of the file:
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@@
 (kicad_sch
-	(version 20231120)
+	(version 20250114)
 	(generator "eeschema")
-	(generator_version "8.0")
+	(generator_version "9.0")
 	(paper "A4")
 	(title_block
@@
 		(comment 2 "Semiconductor\\nionizing radiation detector")
 	)
+	(text "+1.3 mA max"
+		(exclude_from_sim no)
+		(at 242.57 68.58 0)
+		(effects
+			(font
+				(size 1.524 1.524)
+			)
+			(justify left bottom)
+		)
+	)
+	(text "+1.2 mA"
+		(exclude_from_sim no)
+		(at 81.28 74.93 0)
+		(effects
+			(font
+				(size 1.524 1.524)
+			)
+			(justify left bottom)
+		)
+	)
+	(text "73 μA"
+		(exclude_from_sim no)
+		(at 82.55 48.26 0)
+		(effects
+			(font
+				(size 1.524 1.524)
+			)
+			(justify left bottom)
+		)
+	)
+	(text "+1.2 mA"
+		(exclude_from_sim no)
+		(at 83.82 21.59 0)
+		(effects
+			(font
+				(size 1.524 1.524)
+			)
+			(justify left bottom)
+		)
+	)
+	(text "10 μA"
+		(exclude_from_sim no)
+		(at 190.5 118.11 0)
+		(effects
+			(font
+				(size 1.524 1.524)
+			)
+			(justify left bottom)
+		)
+	)
 	(junction
 		(at 29.21 25.4)
@@
 		)
 	)
-	(text "+1.3 mA max"
-		(exclude_from_sim no)
-		(at 242.57 68.58 0)
-		(effects
-			(font
-				(size 1.524 1.524)
-			)
-			(justify left bottom)
-		)
-	)
-	(text "+1.2 mA"
-		(exclude_from_sim no)
-		(at 81.28 74.93 0)
-		(effects
-			(font
-				(size 1.524 1.524)
-			)
-			(justify left bottom)
-		)
-	)
-	(text "73 μA"
-		(exclude_from_sim no)
-		(at 82.55 48.26 0)
-		(effects
-			(font
-				(size 1.524 1.524)
-			)
-			(justify left bottom)
-		)
-	)
-	(text "+1.2 mA"
-		(exclude_from_sim no)
-		(at 83.82 21.59 0)
-		(effects
-			(font
-				(size 1.524 1.524)
-			)
-			(justify left bottom)
-		)
-	)
-	(text "10 μA"
-		(exclude_from_sim no)
-		(at 190.5 118.11 0)
-		(effects
-			(font
-				(size 1.524 1.524)
-			)
-			(justify left bottom)
-		)
-	)
 	(label "VCC3"
 		(at 83.82 52.07 0)
@@
 		(on_board yes)
 		(dnp no)
-		(property "Reference" "TP3"
+		(property "Reference" "TP1"
 			(at 116.84 115.57 0)
 			(effects
@@
 		(on_board yes)
 		(dnp no)
-		(property "Reference" "C2"
+		(property "Reference" "C5"
 			(at 40.64 54.61 0)
 			(effects
@@
 		(on_board yes)
 		(dnp no)
-		(property "Reference" "R11"
+		(property "Reference" "R4"
 			(at 91.44 96.52 90)
 			(effects
@@
 		(on_board yes)
 		(dnp no)
-		(property "Reference" "R11"
+		(property "Reference" "R5"
 			(at 130.81 96.52 90)
 			(effects
@@
 		(on_board yes)
 		(dnp no)
-		(property "Reference" "U3"
+		(property "Reference" "U1"
 			(at 205.74 62.23 0)
 			(effects
@@
 		(on_board yes)
 		(dnp no)
-		(property "Reference" "JP4"
+		(property "Reference" "JP1"
 			(at 236.22 144.78 0)
 			(effects
@@
 		(on_board yes)
 		(dnp no)
-		(property "Reference" "#PWR0152"
+		(property "Reference" "#PWR011"
 			(at 240.03 71.12 0)
 			(effects
@@
 		(on_board yes)
 		(dnp no)
-		(property "Reference" "#PWR0152"
+		(property "Reference" "#PWR02"
 			(at 46.99 25.4 0)
 			(effects
@@
 		(on_board yes)
 		(dnp no)
-		(property "Reference" "C2"
+		(property "Reference" "C1"
 			(at 31.75 29.21 0)
 			(effects
@@
 		(dnp no)
 		(fields_autoplaced yes)
-		(property "Reference" "#PWR024"
+		(property "Reference" "#PWR012"
 			(at 191.77 80.01 0)
 			(effects
@@
 		(on_board yes)
 		(dnp no)
-		(property "Reference" "TP3"
+		(property "Reference" "TP2"
 			(at 227.33 139.7 0)
 			(effects
@@
 		(on_board yes)
 		(dnp no)
-		(property "Reference" "C59"
+		(property "Reference" "C12"
 			(at 261.62 75.1586 0)
 			(effects
@@
 		(on_board yes)
 		(dnp no)
-		(property "Reference" "C59"
+		(property "Reference" "C8"
 			(at 187.96 66.2686 0)
 			(effects
@@
 		(on_board yes)
 		(dnp no)
-		(property "Reference" "R10"
+		(property "Reference" "R7"
 			(at 76.2 109.22 90)
 			(effects
@@
 		(on_board yes)
 		(dnp no)
-		(property "Reference" "C18"
+		(property "Reference" "C15"
 			(at 93.98 85.0392 90)
 			(effects
