File: hw/sch_pcb/USTSIPIN03.kicad_pcb (KiCad board)
At the start: 2 copper layers, 70.6 x 50.3 mm, 100 parts, among them J1 HEADER_2x15, M1 HOLE, M2 HOLE, M3 HOLE, M4 HOLE, M5 RFShield_TwoPieces, Q1 2SK2394-6, U1 ISL21080CIH341Z-TK, U10 ISL21080DIH309, U11 AT24CS64-SSHM, U12 SN74LVC2T45DCU, U13 SN74LVC2T45DCU, U14 SN74LVC2T45DCU, U15 MIC5504-3.3YM5-TR, U2 AD8691, U3 LTC1865-MS, U4 AD8691, U5 SN74LVC2G74, U6 TS3021ILT, U7 SHT31-DIS, U8 OPA314

Commit message: Update production year.
Other:
- board text added: "2026"
- board text removed: "2025"
